Commit message: (feat,to):清理更新train的机器人asset

File: modules/roboparty_train/robolab/data/robots/roboparty/rpo/urdf/rpo_21.urdf (robot description, URDF)
Before this commit: robot rpo_21, 22 links, 21 joints
Links:
- link head_yaw_link: geometry collision mesh filename=../meshes/head_yaw_joint.STL; visual mesh filename=../meshes/head_yaw_joint.STL
- link left_ankle_pitch_link: geometry collision mesh filename=../meshes/left_ankle_pitch_joint.STL; visual mesh filename=../meshes/left_ankle_pitch_joint.STL
- link left_ankle_roll_link: geometry collision mesh filename=../meshes/left_ankle_roll_joint.STL; visual mesh filename=../meshes/left_ankle_roll_joint.STL
- link left_elbow_pitch_link: geometry collision mesh filename=../meshes/left_elbow_pitch_joint.STL; visual mesh filename=../meshes/left_elbow_pitch_joint.STL
- link left_knee_link: geometry collision mesh filename=../meshes/left_knee_joint.STL; visual mesh filename=../meshes/left_knee_joint.STL
- link left_leg_pitch_link: geometry collision mesh filename=../meshes/left_leg_pitch_joint.STL; visual mesh filename=../meshes/left_leg_pitch_joint.STL
- link left_leg_roll_link: geometry collision mesh filename=../meshes/left_leg_roll_joint.STL; visual mesh filename=../meshes/left_leg_roll_joint.STL
- link left_leg_yaw_link: geometry collision mesh filename=../meshes/left_leg_yaw_joint.STL; visual mesh filename=../meshes/left_leg_yaw_joint.STL
- link left_shoulder_pitch_link: geometry collision mesh filename=../meshes/left_shoulder_pitch_joint.STL; visual mesh filename=../meshes/left_shoulder_pitch_joint.STL
- link left_shoulder_roll_link: geometry collision mesh filename=../meshes/left_shoulder_roll_joint.STL; visual mesh filename=../meshes/left_shoulder_roll_joint.STL
- link left_shoulder_yaw_link: geometry collision mesh filename=../meshes/left_shoulder_yaw_joint.STL; visual mesh filename=../meshes/left_shoulder_yaw_joint.STL
- link right_ankle_pitch_link: geometry collision mesh filename=../meshes/right_ankle_pitch_joint.STL; visual mesh filename=../meshes/right_ankle_pitch_joint.STL
- link right_ankle_roll_link: geometry collision mesh filename=../meshes/right_ankle_roll_joint.STL; visual mesh filename=../meshes/right_ankle_roll_joint.STL
- link right_elbow_pitch_link: geometry collision mesh filename=../meshes/right_elbow_pitch_joint.STL; visual mesh filename=../meshes/right_elbow_pitch_joint.STL
- link right_knee_link: geometry collision mesh filename=../meshes/right_knee_joint.STL; visual mesh filename=../meshes/right_knee_joint.STL
- link right_leg_pitch_link: geometry collision mesh filename=../meshes/right_leg_pitch_joint.STL; visual mesh filename=../meshes/right_leg_pitch_joint.STL
- link right_leg_roll_link: geometry collision mesh filename=../meshes/right_leg_roll_joint.STL; visual mesh filename=../meshes/right_leg_roll_joint.STL
- link right_leg_yaw_link: geometry collision mesh filename=../meshes/right_leg_yaw_joint.STL; visual mesh filename=../meshes/right_leg_yaw_joint.STL
- link right_shoulder_pitch_link: geometry collision mesh filename=../meshes/right_shoulder_pitch_joint.STL; visual mesh filename=../meshes/right_shoulder_pitch_joint.STL
- link right_shoulder_roll_link: geometry collision mesh filename=../meshes/right_shoulder_roll_joint.STL; visual mesh filename=../meshes/right_shoulder_roll_joint.STL
- link right_shoulder_yaw_link: geometry collision mesh filename=../meshes/right_shoulder_yaw_joint.STL; visual mesh filename=../meshes/right_shoulder_yaw_joint.STL

Commit message: fix(deploy,rl)：导入了新的urdf以及修改了手柄空数组的问题，现在能正常启动了

File: modules/roboparty_train/robolab/data/robots/roboparty/rpo/urdf/rpo_21.urdf (robot description, URDF)
Before this commit: robot rpo_21, 22 links, 21 joints
Links:
- link base_link: mass 7.23135683 -> 7.31425690; geometry collision box size=0.16 0.16 0.206; collision box size=0.162 0.635 0.09
- link head_yaw_link: mass 0.82067000 -> 4.43676000; geometry collision box size=0.591 0.578 0.661; visual mesh filename=../meshes/head_yaw_joint.STL
- link left_ankle_pitch_link: geometry visual mesh filename=../meshes/left_ankle_pitch_joint.STL
- link left_elbow_pitch_link: mass 0.42600716 -> 0.48283833; geometry collision cylinder length=0.344 radius=0.055; visual mesh filename=../meshes/left_elbow_pitch_joint.STL
- link left_knee_link: geometry collision box size=0.109 0.1 0.272; visual mesh filename=../meshes/left_knee_joint.STL
- link left_leg_pitch_link: geometry visual mesh filename=../meshes/left_leg_pitch_joint.STL
- link left_leg_roll_link: geometry collision box size=0.147 0.12 0.171; visual mesh filename=../meshes/left_leg_roll_joint.STL
- link left_leg_yaw_link: geometry collision box size=0.12 0.101 0.184; visual mesh filename=../meshes/left_leg_yaw_joint.STL
- link left_shoulder_pitch_link: mass 0.29250686 -> 0.30923666; geometry visual mesh filename=../meshes/left_shoulder_pitch_joint.STL
- link left_shoulder_roll_link: mass 0.46031769 -> 0.44708769; geometry visual mesh filename=../meshes/left_shoulder_roll_joint.STL
- link left_shoulder_yaw_link: mass 0.74847871 -> 0.73732871; geometry collision cylinder length=0.139 radius=0.068; visual mesh filename=../meshes/left_shoulder_yaw_joint.STL
- link right_ankle_pitch_link: geometry visual mesh filename=../meshes/right_ankle_pitch_joint.STL
- link right_ankle_roll_link: mass 1.46135369 -> 1.46424250
- link right_elbow_pitch_link: mass 0.42436129 -> 0.48283833; geometry collision cylinder length=0.344 radius=0.055; visual mesh filename=../meshes/right_elbow_pitch_joint.STL
- link right_knee_link: geometry collision box size=0.109 0.1 0.272; visual mesh filename=../meshes/right_knee_joint.STL
- link right_leg_pitch_link: geometry visual mesh filename=../meshes/right_leg_pitch_joint.STL
- link right_leg_roll_link: geometry collision box size=0.147 0.12 0.171; visual mesh filename=../meshes/right_leg_roll_joint.STL
- link right_leg_yaw_link: geometry collision box size=0.12 0.101 0.184; visual mesh filename=../meshes/right_leg_yaw_joint.STL
- link right_shoulder_pitch_link: mass 0.29250686 -> 0.30923666; geometry visual mesh filename=../meshes/right_shoulder_pitch_joint.STL
- link right_shoulder_roll_link: mass 0.46031769 -> 0.44708769; geometry visual mesh filename=../meshes/right_shoulder_roll_joint.STL
- link right_shoulder_yaw_link: mass 0.74847871 -> 0.73732871; geometry collision cylinder length=0.139 radius=0.068; visual mesh filename=../meshes/right_shoulder_yaw_joint.STL
Joints:
- joint left_ankle_pitch_joint: origin xyz=0 0.052 -0.21369 rpy=0 0 0 -> xyz=0 0.0510000000000015 -0.213694214876033 rpy=0 0 0
- joint left_knee_joint: origin xyz=6.00000000000895E-05 -0.0510000000000023 -0.0899000000000003 rpy=0 0 0 -> xyz=6.00000000000427E-05 -0.0509999999999998 -0.0970000000000002 rpy=0 0 0
- joint left_leg_yaw_joint: origin xyz=0.0629500000000003 -5.99999999965073E-05 -0.129000000000001 rpy=0 0 0 -> xyz=0.0629500000000003 -5.99999999991163E-05 -0.122000000000002 rpy=0 0 0
- joint right_ankle_pitch_joint: origin xyz=0 -0.0509999999999989 -0.213694214876033 rpy=0 0 0 -> xyz=0 -0.051 -0.21369 rpy=0 0 0
- joint right_knee_joint: origin xyz=6.00000000000149E-05 0.0510000000000006 -0.0969999999999999 rpy=0 0 0 -> xyz=6E-05 0.051 -0.097 rpy=0 0 0
- joint right_leg_pitch_joint: origin xyz=0 -0.0709999999999998 -0.0630000000000002 rpy=0 0 0 -> xyz=0 -0.071 -0.063 rpy=0 0 0
- joint right_leg_roll_joint: origin xyz=-0.051 -0.0969 -6E-05 rpy=0 0 0 -> xyz=-0.0509999999999999 -0.0969999999999997 -6.00000000014755E-05 rpy=0 0 0
