Commit message: feat(rpo): 更新 Loobot722 关节限位和电机参数
- 写入实测关节位置限位
- 更新耦合踝关节安全范围
- 按 DM 官方参数更新 effort 和 velocity
- 同步所有策略配置的 joint_limits

File: modules/roboparty_train/robolab/data/robots/roboparty/rpo/urdf/Loobot722.urdf (robot description, URDF)
Before this commit: robot Loobot722, 22 links, 21 joints
Joints:
- joint head_yaw_joint: limit lower=-2 upper=2 effort=250 velocity=12 -> lower=-1.510834 upper=1.630999 effort=27 velocity=10.471976
- joint left_ankle_pitch_joint: limit lower=-2 upper=2 effort=250 velocity=12 -> lower=-0.2880 upper=0.0790 effort=97 velocity=6.283185
- joint left_ankle_roll_joint: limit lower=-2 upper=2 effort=250 velocity=12 -> lower=-0.0415 upper=0.1290 effort=97 velocity=6.283185
- joint left_elbow_pitch_joint: limit lower=-2 upper=2 effort=250 velocity=12 -> lower=0 upper=1.576829 effort=27 velocity=10.471976
- joint left_knee_joint: limit lower=-2 upper=2 effort=250 velocity=12 -> lower=-0.171092 upper=1.855307 effort=120 velocity=20.943951
- joint left_leg_pitch_joint: limit lower=-2 upper=2 effort=150 velocity=12 -> lower=-1.445220 upper=0.493057 effort=120 velocity=20.943951
- joint left_leg_roll_joint: limit lower=-2 upper=2 effort=250 velocity=12 -> lower=-0.382429 upper=0.689517 effort=120 velocity=20.943951
- joint left_leg_yaw_joint: limit lower=-2 upper=2 effort=250 velocity=12 -> lower=-0.852707 upper=0.862707 effort=120 velocity=20.943951
- joint left_shoulder_pitch_joint: limit lower=-2 upper=2 effort=250 velocity=12 -> lower=-2.984856 upper=1.637865 effort=27 velocity=10.471976
- joint left_shoulder_roll_joint: limit lower=-2 upper=2 effort=250 velocity=12 -> lower=0.037576 upper=2.176890 effort=27 velocity=10.471976
- joint left_shoulder_yaw_joint: limit lower=-2 upper=2 effort=250 velocity=12 -> lower=-1.550889 upper=1.605822 effort=27 velocity=10.471976
- joint right_ankle_pitch_joint: limit lower=-2 upper=2 effort=250 velocity=12 -> lower=-0.2745 upper=0.1380 effort=97 velocity=6.283185
- joint right_ankle_roll_joint: limit lower=-2 upper=2 effort=250 velocity=12 -> lower=-0.1080 upper=0.0805 effort=97 velocity=6.283185
- joint right_elbow_pitch_joint: limit lower=-2 upper=2 effort=250 velocity=12 -> lower=0 upper=1.584840 effort=27 velocity=10.471976
- joint right_knee_joint: limit lower=-2 upper=2 effort=250 velocity=12 -> lower=0.061608 upper=1.811818 effort=120 velocity=20.943951
- joint right_leg_pitch_joint: limit lower=-2 upper=2 effort=250 velocity=12 -> lower=-1.444076 upper=0.485809 effort=120 velocity=20.943951
- joint right_leg_roll_joint: limit lower=-2 upper=2 effort=250 velocity=12 -> lower=-0.700198 upper=0.382048 effort=120 velocity=20.943951
- joint right_leg_yaw_joint: limit lower=-2 upper=2 effort=250 velocity=12 -> lower=-0.858130 upper=0.869574 effort=120 velocity=20.943951
- joint right_shoulder_pitch_joint: limit lower=-2 upper=2 effort=250 velocity=12 -> lower=-3.385023 upper=1.647783 effort=27 velocity=10.471976
- joint right_shoulder_roll_joint: limit lower=-2 upper=2 effort=250 velocity=12 -> lower=-2.210078 upper=0 effort=27 velocity=10.471976
- joint right_shoulder_yaw_joint: limit lower=-2 upper=2 effort=250 velocity=12 -> lower=-1.594759 upper=1.635576 effort=27 velocity=10.471976
