Commit message: fix(deploy,rpo): 完善实机启动与策略切换保护
- 固定 USB-CAN 映射并在启动前校验四路 CAN 状态
- 从实时关节姿态平滑接入策略
- 暂停策略后平滑进入并持续保持安全站姿
- 为关节反馈越界增加测量容差及 CAN/ID 诊断
- 修正右膝和左肩 roll 零点限位并同步训练与部署 URDF
- 更新手柄控制和实机验证文档

File: modules/roboparty_deploy/src/inference/robots/rpo/description/urdf/Loobot722.urdf (robot description, URDF)
Before this commit: robot Loobot722, 22 links, 21 joints
Joints:
- joint left_shoulder_roll_joint: limit lower=0.037576 upper=2.176890 effort=27 velocity=10.471976 -> lower=0 upper=2.176890 effort=27 velocity=10.471976
- joint right_knee_joint: limit lower=0.061608 upper=1.811818 effort=120 velocity=20.943951 -> lower=0 upper=1.811818 effort=120 velocity=20.943951

Commit message: fix(deploy,rpo):重新确认了新的urdf上下限和方向

File: modules/roboparty_deploy/src/inference/robots/rpo/description/urdf/Loobot722.urdf (robot description, URDF)
Before this commit: robot Loobot722, 22 links, 21 joints
Joints:
- joint left_ankle_pitch_joint: limit lower=-0.2880 upper=0.0790 effort=97 velocity=6.283185 -> lower=-0.377162 upper=0.357987 effort=97 velocity=6.283185
- joint left_ankle_roll_joint: limit lower=-0.0415 upper=0.1290 effort=97 velocity=6.283185 -> lower=-0.589145 upper=0.520970 effort=97 velocity=6.283185
- joint left_elbow_pitch_joint: limit lower=0 upper=1.576829 effort=27 velocity=10.471976 -> lower=-1.576829 upper=0 effort=27 velocity=10.471976
- joint right_ankle_pitch_joint: limit lower=-0.2745 upper=0.1380 effort=97 velocity=6.283185 -> lower=-0.450025 upper=0.372177 effort=97 velocity=6.283185
- joint right_ankle_roll_joint: limit lower=-0.1080 upper=0.0805 effort=97 velocity=6.283185 -> lower=-0.520970 upper=0.890271 effort=97 velocity=6.283185
- joint right_elbow_pitch_joint: limit lower=0 upper=1.584840 effort=27 velocity=10.471976 -> lower=-1.584840 upper=0 effort=27 velocity=10.471976
